Commit message: changes

File: legged_lab/assets/Robot3/urdf/Robot3.urdf (robot description, URDF)
Before this commit: robot Robot3, 32 links, 31 joints
Links:
- link imu_in_torso_link: mass 0 -> 0.01
- link left_ankle_pitch_link: mass 0.07 -> 0.11
- link left_ankle_roll_link: mass 1.158 -> 1.166
- link left_hip_pitch_link: mass 3.03 -> 3.12
- link left_hip_roll_link: mass 3.08 -> 1.783
- link left_hip_yaw_link: mass 5.5 -> 5.44
- link left_knee_link: mass 3.67 -> 3.85
- link left_shoulder_pitch_link: mass 1.2641752 -> 2.525
- link left_shoulder_yaw_link: mass 2.2112 -> 2.21
- link pelvis: mass 10.304 -> 10.775
- link right_ankle_pitch_link: mass 0.7 -> 0.11
- link right_ankle_roll_link: mass 1.158 -> 1.166
- link right_hip_pitch_link: mass 3.03 -> 3.12
- link right_hip_roll_link: mass 3.08 -> 1.783
- link right_hip_yaw_link: mass 5.5 -> 5.44
- link right_knee_link: mass 3.67 -> 3.85; geometry collision cylinder length=0.25 radius=0.05; visual mesh filename=../meshes/right_knee_link.STL
- link right_shoulder_pitch_link: mass 1.2641751 -> 2.525
- link right_shoulder_yaw_link: mass 2.2111852 -> 2.21
- link waist_yaw_link: mass 6.84 -> 17.7
Joints:
- joint head_pitch_joint: limit lower=-0.5235988 upper=0.5235988 effort=4.8 velocity=4.712 -> lower=-0.5235988 upper=0.5235988 effort=3.3 velocity=12.36
- joint head_roll_joint: limit lower=-0.5235988 upper=0.5235988 effort=4.8 velocity=4.712 -> lower=-0.5235988 upper=0.5235988 effort=3.3 velocity=12.36
- joint head_yaw_joint: limit lower=-2.7925268 upper=2.7925268 effort=4.8 velocity=4.712 -> lower=-2.7925268 upper=2.7925268 effort=3.3 velocity=12.36
- joint left_ankle_pitch_joint: limit lower=-0.925 upper=0.925 effort=90 velocity=16 -> lower=-0.916 upper=0.488 effort=90 velocity=16
- joint left_ankle_roll_joint: limit lower=-0.349 upper=0.349 effort=90 velocity=16 -> lower=-0.35 upper=0.35 effort=90 velocity=16
- joint left_elbow_joint: axis 0 -1 0 -> 0 1 0; limit lower=0 upper=2.2340214 effort=108 velocity=4 -> lower=-2.2340214 upper=0 effort=108 velocity=4
- joint left_hip_roll_joint: axis -1 0 0 -> 1 0 0; limit lower=-2.094 upper=0.436 effort=320 velocity=10.47 -> lower=-0.436 upper=2.094 effort=320 velocity=10.47
- joint left_shoulder_pitch_joint: axis 0 -1 0 -> 0 1 0; limit lower=-3.1066861 upper=3.1066861 effort=194 velocity=2.82744 -> lower=-3.1066861 upper=3.1066861 effort=194 velocity=3.77
- joint left_shoulder_roll_joint: limit lower=-0.3141593 upper=3.1066861 effort=194 velocity=2.8744 -> lower=-0.4363323 upper=3.1066861 effort=194 velocity=3.77
- joint left_shoulder_yaw_joint: limit lower=-3.1066861 upper=3.1066861 effort=102 velocity=3.1416 -> lower=-3.1066861 upper=3.1066861 effort=102 velocity=4.19
- joint left_wrist_pitch_joint: axis 0 -1 0 -> 0 1 0
- joint left_wrist_roll_joint: axis 0 0 -1 -> 0 0 1; limit lower=-3.1066861 upper=3.1066861 effort=66 velocity=3.56 -> lower=-3.1066861 upper=3.1066861 effort=66 velocity=4.29
- joint left_wrist_yaw_joint: axis -1 0 0 -> 1 0 0
- joint right_ankle_pitch_joint: axis 0 -1 0 -> 0 1 0; limit lower=-0.925 upper=0.925 effort=90 velocity=16 -> lower=-0.916 upper=0.488 effort=90 velocity=16
- joint right_elbow_joint: axis 0 -1 0 -> 0 1 0; limit lower=0 upper=2.2340214 effort=108 velocity=4 -> lower=-2.2340214 upper=0 effort=108 velocity=4
- joint right_hip_pitch_joint: axis 0 -1 0 -> 0 1 0
- joint right_knee_joint: axis 0 -1 0 -> 0 1 0; limit lower=-2.356 upper=0 effort=450 velocity=6.8 -> lower=0 upper=2.356 effort=450 velocity=6.8
- joint right_shoulder_pitch_joint: limit lower=-3.1066861 upper=3.1066861 effort=194 velocity=2.82744 -> lower=-3.1066861 upper=3.1066861 effort=194 velocity=3.77
- joint right_shoulder_roll_joint: limit lower=-3.1066861 upper=0.4363323 effort=194 velocity=2.82744 -> lower=-3.1066861 upper=0.4363323 effort=194 velocity=3.77
- joint right_shoulder_yaw_joint: limit lower=-3.1066861 upper=3.1066861 effort=102 velocity=3.1416 -> lower=-3.1066861 upper=3.1066861 effort=102 velocity=4.19
- joint right_wrist_pitch_joint: limit lower=-1.3089969 upper=1.3089969 effort=60 velocity=3.5 -> lower=-1.309 upper=1.309 effort=60 velocity=3.5
- joint right_wrist_roll_joint: axis 0 0 -1 -> 0 0 1; limit lower=-3.1066861 upper=3.1066861 effort=66 velocity=3.56 -> lower=-3.1066861 upper=3.1066861 effort=66 velocity=4.29
- joint right_wrist_yaw_joint: axis -1 0 0 -> 1 0 0
- joint waist_yaw_joint: axis 0 0 -1 -> 0 0 1

Commit message: changes

File: legged_lab/assets/Robot3/urdf/Robot3.urdf (robot description, URDF)
Before this commit: robot Robot3, 32 links, 31 joints
Joints:
- joint head_pitch_joint: limit lower=-0.5235988 upper=0.5235988 effort=3.3 velocity=12.36 -> lower=-0.5235988 upper=0.5235988 effort=4.8 velocity=6.18
- joint head_roll_joint: limit lower=-0.5235988 upper=0.5235988 effort=3.3 velocity=12.36 -> lower=-0.5235988 upper=0.5235988 effort=4.8 velocity=6.18
- joint head_yaw_joint: limit lower=-2.7925268 upper=2.7925268 effort=3.3 velocity=12.36 -> lower=-2.7925268 upper=2.7925268 effort=4.8 velocity=6.18
- joint left_ankle_pitch_joint: limit lower=-0.916 upper=0.488 effort=90 velocity=16 -> lower=-0.916 upper=0.488 effort=70 velocity=18.43
- joint left_ankle_roll_joint: limit lower=-0.35 upper=0.35 effort=90 velocity=16 -> lower=-0.35 upper=0.35 effort=70 velocity=18.43
- joint left_elbow_joint: limit lower=-2.2340214 upper=0 effort=108 velocity=4 -> lower=-2.2340214 upper=0 effort=5000 velocity=4
- joint left_hip_pitch_joint: limit lower=-2.618 upper=2.618 effort=450 velocity=6.8 -> lower=-2.618 upper=2.618 effort=450 velocity=7.54
- joint left_hip_roll_joint: limit lower=-0.436 upper=2.094 effort=320 velocity=10.47 -> lower=-0.436 upper=2.094 effort=320 velocity=13.09
- joint left_hip_yaw_joint: limit lower=-2.618 upper=2.618 effort=120 velocity=13.299 -> lower=-2.618 upper=2.618 effort=120 velocity=16.55
- joint left_knee_joint: limit lower=0 upper=2.356 effort=450 velocity=6.8 -> lower=0 upper=2.356 effort=320 velocity=13.09
- joint left_shoulder_pitch_joint: limit lower=-3.1066861 upper=3.1066861 effort=194 velocity=3.77 -> lower=-3.1066861 upper=3.1066861 effort=207 velocity=3.14
- joint left_shoulder_roll_joint: limit lower=-0.4363323 upper=3.1066861 effort=194 velocity=3.77 -> lower=-0.4363323 upper=3.1066861 effort=207 velocity=3.14
- joint left_wrist_pitch_joint: limit lower=-1.309 upper=1.309 effort=60 velocity=3.5 -> lower=-1.309 upper=1.309 effort=600 velocity=3.5
- joint left_wrist_yaw_joint: limit lower=-0.5235988 upper=0.5235988 effort=60 velocity=3.5 -> lower=-0.5235988 upper=0.5235988 effort=600 velocity=3.5
- joint right_ankle_pitch_joint: limit lower=-0.916 upper=0.488 effort=90 velocity=16 -> lower=-0.916 upper=0.488 effort=70 velocity=18.43
- joint right_ankle_roll_joint: limit lower=-0.35 upper=0.35 effort=90 velocity=16 -> lower=-0.35 upper=0.35 effort=70 velocity=18.43
- joint right_elbow_joint: limit lower=-2.2340214 upper=0 effort=108 velocity=4 -> lower=-2.2340214 upper=0 effort=5000 velocity=4
- joint right_hip_pitch_joint: limit lower=-2.618 upper=2.618 effort=450 velocity=6.8 -> lower=-2.618 upper=2.618 effort=450 velocity=7.54
- joint right_hip_roll_joint: limit lower=-2.094 upper=0.436 effort=320 velocity=10.47 -> lower=-2.094 upper=0.436 effort=320 velocity=13.09
- joint right_hip_yaw_joint: limit lower=-2.618 upper=2.618 effort=120 velocity=13.299 -> lower=-2.618 upper=2.618 effort=120 velocity=16.55
- joint right_knee_joint: limit lower=0 upper=2.356 effort=450 velocity=6.8 -> lower=0 upper=2.356 effort=320 velocity=13.09
- joint right_shoulder_pitch_joint: limit lower=-3.1066861 upper=3.1066861 effort=194 velocity=3.77 -> lower=-3.1066861 upper=3.1066861 effort=207 velocity=3.14
- joint right_shoulder_roll_joint: limit lower=-3.1066861 upper=0.4363323 effort=194 velocity=3.77 -> lower=-3.1066861 upper=0.4363323 effort=207 velocity=3.14
- joint right_wrist_pitch_joint: limit lower=-1.309 upper=1.309 effort=60 velocity=3.5 -> lower=-1.309 upper=1.309 effort=600 velocity=3.5
- joint right_wrist_yaw_joint: limit lower=-0.5235988 upper=0.5235988 effort=60 velocity=3.5 -> lower=-0.5235988 upper=0.5235988 effort=600 velocity=3.5
- joint waist_yaw_joint: limit lower=-2.6005406 upper=2.6005406 effort=200 velocity=7.75 -> lower=-2.6005406 upper=2.6005406 effort=200 velocity=8.38
